File: doc/boards/pixelix/v2.1/pixelix.kicad_sch (KiCad schematic)
At the start: 25 parts

Commit message: Update file kicad
Parts:
- removed J: USB_C_Receptacle_USB2.0, symbol Connector:USB_C_Receptacle_USB2.0
- removed U (x8): (no value), symbol esp32bb-rescue:C-esp32bb-rescue
- removed U (x6): (no value), symbol esp32bb-rescue:R-esp32bb-rescue
- removed U: CP2102N-Axx-xQFN28, Package_DFN_QFN:QFN-28-1EP_5x5mm_P0.5mm_EP3.35x3.35mm, symbol Interface_USB:CP2102N-Axx-xQFN28
- removed U (x2): (no value), symbol esp32bb-rescue:SWITCH_SPST-esp32bb-rescue
- removed U (x2): (no value), symbol esp32bb-rescue:D-esp32bb-rescue
- removed U: (no value), symbol esp32bb-rescue:NCP1117ST33T3G-esp32bb-rescue
- removed U (x2): (no value), symbol esp32bb-rescue:MMBT3904-esp32bb-rescue
- added H (x5): MountingHole, symbol Mechanical:MountingHole
- added U (x2): (no value), symbol esp32bb-rescue:C-esp32bb-rescue
- added U (x2): (no value), symbol esp32bb-rescue:SWITCH_SPST-esp32bb-rescue
- added U: (no value), symbol esp32bb-rescue:R-esp32bb-rescue
Connections:
- net EN: now also U.1, U.1
- net GND: now also U.2, U.2, U.2, U.2
- net IO0(boot): now also U.1, U.1
- net IO5: now also U.1
- net at U.2 (A): now also U.2
Other:
- added sheet CH340G (CH340G.kicad_sch)
- added sheet WS2812B (WS2812B_matrix.kicad_sch)
